File: currentlim.sch (EAGLE design)
At the start: 13 parts

Commit message: relay n stuff
Parts:
- added C3, C4: (no value), rcl:CPOL-USE2.5-6
- added D1: 1N5060GP, diode:1N5060GP
- added POWER: (no value), pinhead:PINHD-1X2
- added U$3: JD2912, currentlim:JD2912
- added U$4, U$5: XT90_ST, XT Connectors:XT90_ST
- added U$6: LM1117MPX-3.3/NOPB, currentlim:LM1117MPX-3.3/NOPB
Connections:
- net N$3 renamed RESET
- removed net OC: JP1.3
- new net +12V: C3.+, D1.A, POWER.1, U$3G$1.1, U$6.VIN
- new net N$4: U$2.IP-, U$5.V+
- new net N$5: U$2.IP+, U$3G$2.P
- new net N$6: U$3G$2.O, U$4.V-
- new net N$7: U$4.V+, U$5.V-
- new net N$8: D1.C, T1.C, U$3G$1.2
- net +3V3: now also C4.+, U$6.VOUT
- net GND: now also C3.-, C4.-, POWER.2, U$6.ADJ
- net OC_DETECT: now also JP1.3
