File: currentsense.sch (EAGLE design)
At the start: 18 parts

Commit message: more layout work
Connections:
- net N$1 renamed M-IP+
- net N$3 renamed M-IP-
- net N$4 renamed M+
- removed net OC_DETECT: DATA.3
- removed net SDA: DATA.1
- net OC_DETECT/6: now also DATA.2
- net SCL/7: now also DATA.3; no longer DATA.2
- net SDA/5: now also DATA.1
Changed lines of the file:
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@@
-</segment>
-<segment>
-<pinref part="DATA" gate="A" pin="2"/>
-<wire x1="72.39" y1="29.21" x2="63.5" y2="29.21" width="0.1524" layer="91"/>
-<label x="63.5" y="29.21" size="1.27" layer="95" rot="R180" xref="yes"/>
 </segment>
 <segment>
@@
 <label x="91.44" y="93.98" size="1.27" layer="95" rot="R180" xref="yes"/>
 </segment>
-</net>
-<net name="SDA" class="0">
-<segment>
-<pinref part="DATA" gate="A" pin="1"/>
-<wire x1="72.39" y1="31.75" x2="63.5" y2="31.75" width="0.1524" layer="91"/>
-<label x="63.5" y="31.75" size="1.27" layer="95" rot="R180" xref="yes"/>
+<segment>
+<pinref part="DATA" gate="A" pin="3"/>
+<wire x1="72.39" y1="26.67" x2="63.5" y2="26.67" width="0.1524" layer="91"/>
+<label x="63.5" y="26.67" size="1.27" layer="95" rot="R180" xref="yes"/>
 </segment>
 </net>
@@
 </segment>
 </net>
-<net name="OC_DETECT" class="0">
-<segment>
-<pinref part="DATA" gate="A" pin="3"/>
-<wire x1="72.39" y1="26.67" x2="63.5" y2="26.67" width="0.1524" layer="91"/>
-<label x="63.5" y="26.67" size="1.27" layer="95" rot="R180" xref="yes"/>
-</segment>
-</net>
 <net name="CURRENT" class="0">
 <segment>
@@
 </segment>
 </net>
-<net name="N$1" class="0">
+<net name="M-IP+" class="0">
 <segment>
 <pinref part="U$4" gate="G$1" pin="V-"/>
@@
 <wire x1="-24.384" y1="82.296" x2="-24.384" y2="62.23" width="0.1524" layer="91"/>
 <wire x1="-24.384" y1="62.23" x2="-8.89" y2="62.23" width="0.1524" layer="91"/>
-</segment>
-</net>
-<net name="N$3" class="0">
+<label x="-22.86" y="68.58" size="1.778" layer="95" xref="yes"/>
+</segment>
+</net>
+<net name="M-IP-" class="0">
 <segment>
 <pinref part="U$2" gate="G$1" pin="IP-"/>
@@
 <wire x1="-36.322" y1="56.896" x2="-8.89" y2="56.896" width="0.1524" layer="91"/>
 <wire x1="-8.89" y1="56.896" x2="-8.89" y2="57.15" width="0.1524" layer="91"/>
+<label x="-22.86" y="55.88" size="1.778" layer="95" rot="R270" xref="yes"/>
 </segment>
 </net>
@@
 <label x="111.76" y="93.98" size="1.27" layer="95" xref="yes"/>
 </segment>
+<segment>
+<pinref part="DATA" gate="A" pin="1"/>
+<wire x1="72.39" y1="31.75" x2="63.5" y2="31.75" width="0.1524" layer="91"/>
+<label x="63.5" y="31.75" size="1.27" layer="95" rot="R180" xref="yes"/>
+</segment>
 </net>
 <net name="OC_DETECT/6" class="0">
@@
 <label x="91.44" y="96.52" size="1.27" layer="95" rot="R180" xref="yes"/>
 </segment>
-</net>
-<net name="N$4" class="0">
+<segment>
+<pinref part="DATA" gate="A" pin="2"/>
+<wire x1="72.39" y1="29.21" x2="63.5" y2="29.21" width="0.1524" layer="91"/>
+<label x="63.5" y="29.21" size="1.27" layer="95" rot="R180" xref="yes"/>
+</segment>
+</net>
+<net name="M+" class="0">
 <segment>
 <pinref part="U$5" gate="G$1" pin="V+"/>
@@
 <wire x1="-36.322" y1="61.976" x2="-29.464" y2="61.976" width="0.1524" layer="91"/>
 <wire x1="-29.464" y1="61.976" x2="-29.464" y2="82.296" width="0.1524" layer="91"/>
-</segment>
-</net>
+<label x="-30.48" y="71.12" size="1.778" layer="95" rot="R180" xref="yes"/>
+</segment>
+</net>

Commit message: add board files
Parts:
- added C5, C6: 0.1uF, rcl:C-USC0805
- C1, C2: value (none) -> 0.1uF
- C3, C4: value (none) -> 10uF
- R2, R3: value (none) -> 10k
- R6: value (none) -> 2.2k
Connections:
- net +3V3: now also C5.1
- net CURRENT: now also U$1.PB4/XTAL2/CLKO/ADC2; no longer U$1.PB3/XTAL1/CLKI/ADC3
- net GND: now also C5.2, C6.2
- net TEMPERATURE: now also C6.1, U$1.PB3/XTAL1/CLKI/ADC3; no longer U$1.PB4/XTAL2/CLKO/ADC2
Changed lines of the file:
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@@
 <class number="0" name="default" width="0" drill="0">
+</class>
+<class number="1" name="hicurrent" width="0" drill="0">
+<clearance class="1" value="0.762"/>
 </class>
 </classes>
@@
 <part name="U$1" library="currentlim" deviceset="ATTINY85" device="V-10SUR"/>
 <part name="U$2" library="currentlim" deviceset="ACS781" device="LLRTR-050B-T_M"/>
-<part name="R3" library="rcl" library_urn="urn:adsk.eagle:library:334" deviceset="R-US_" device="M0805" package3d_urn="urn:adsk.eagle:package:23556/2"/>
+<part name="R3" library="rcl" library_urn="urn:adsk.eagle:library:334" deviceset="R-US_" device="M0805" package3d_urn="urn:adsk.eagle:package:23556/2" value="10k"/>
 <part name="+3V1" library="supply1" library_urn="urn:adsk.eagle:library:371" deviceset="+3V3" device=""/>
 <part name="GND1" library="supply1" library_urn="urn:adsk.eagle:library:371" deviceset="GND" device=""/>
-<part name="R2" library="rcl" library_urn="urn:adsk.eagle:library:334" deviceset="R-US_" device="M0805" package3d_urn="urn:adsk.eagle:package:23556/2"/>
+<part name="R2" library="rcl" library_urn="urn:adsk.eagle:library:334" deviceset="R-US_" device="M0805" package3d_urn="urn:adsk.eagle:package:23556/2" value="10k"/>
 <part name="+3V2" library="supply1" library_urn="urn:adsk.eagle:library:371" deviceset="+3V3" device=""/>
 <part name="+3V3" library="supply1" library_urn="urn:adsk.eagle:library:371" deviceset="+3V3" device=""/>
@@
 <part name="GND4" library="supply1" library_urn="urn:adsk.eagle:library:371" deviceset="GND" device=""/>
 <part name="DATA" library="pinhead" library_urn="urn:adsk.eagle:library:325" deviceset="PINHD-1X3" device="" package3d_urn="urn:adsk.eagle:package:22458/2"/>
-<part name="R6" library="rcl" library_urn="urn:adsk.eagle:library:334" deviceset="R-US_" device="M0805" package3d_urn="urn:adsk.eagle:package:23556/2"/>
-<part name="C1" library="rcl" library_urn="urn:adsk.eagle:library:334" deviceset="C-US" device="C0805" package3d_urn="urn:adsk.eagle:package:23617/2"/>
-<part name="C2" library="rcl" library_urn="urn:adsk.eagle:library:334" deviceset="C-US" device="C0805" package3d_urn="urn:adsk.eagle:package:23617/2"/>
+<part name="R6" library="rcl" library_urn="urn:adsk.eagle:library:334" deviceset="R-US_" device="M0805" package3d_urn="urn:adsk.eagle:package:23556/2" value="2.2k"/>
+<part name="C1" library="rcl" library_urn="urn:adsk.eagle:library:334" deviceset="C-US" device="C0805" package3d_urn="urn:adsk.eagle:package:23617/2" value="0.1uF"/>
+<part name="C2" library="rcl" library_urn="urn:adsk.eagle:library:334" deviceset="C-US" device="C0805" package3d_urn="urn:adsk.eagle:package:23617/2" value="0.1uF"/>
 <part name="U$4" library="XT Connectors" deviceset="XT60-RA" device=""/>
 <part name="U$5" library="XT Connectors" deviceset="XT60-RA" device=""/>
@@
 <part name="+3V5" library="supply1" library_urn="urn:adsk.eagle:library:371" deviceset="+3V3" device=""/>
 <part name="GND6" library="supply1" library_urn="urn:adsk.eagle:library:371" deviceset="GND" device=""/>
-<part name="C3" library="rcl" library_urn="urn:adsk.eagle:library:334" deviceset="CPOL-US" device="E2.5-6" package3d_urn="urn:adsk.eagle:package:23349/1"/>
-<part name="C4" library="rcl" library_urn="urn:adsk.eagle:library:334" deviceset="CPOL-US" device="E2.5-6" package3d_urn="urn:adsk.eagle:package:23349/1"/>
+<part name="C3" library="rcl" library_urn="urn:adsk.eagle:library:334" deviceset="CPOL-US" device="E2.5-6" package3d_urn="urn:adsk.eagle:package:23349/1" value="10uF"/>
+<part name="C4" library="rcl" library_urn="urn:adsk.eagle:library:334" deviceset="CPOL-US" device="E2.5-6" package3d_urn="urn:adsk.eagle:package:23349/1" value="10uF"/>
 <part name="P+1" library="supply1" library_urn="urn:adsk.eagle:library:371" deviceset="VCC" device=""/>
 <part name="P+2" library="supply1" library_urn="urn:adsk.eagle:library:371" deviceset="VCC" device=""/>
@@
 <part name="R1" library="rcl" library_urn="urn:adsk.eagle:library:334" deviceset="R-US_" device="M0805" package3d_urn="urn:adsk.eagle:package:23556/2" value="10k"/>
 <part name="+3V7" library="supply1" library_urn="urn:adsk.eagle:library:371" deviceset="+3V3" device=""/>
+<part name="C5" library="rcl" library_urn="urn:adsk.eagle:library:334" deviceset="C-US" device="C0805" package3d_urn="urn:adsk.eagle:package:23617/2" value="0.1uF"/>
+<part name="C6" library="rcl" library_urn="urn:adsk.eagle:library:334" deviceset="C-US" device="C0805" package3d_urn="urn:adsk.eagle:package:23617/2" value="0.1uF"/>
 </parts>
 <sheets>
@@
 <attribute name="VALUE" x="154.432" y="73.66" size="1.778" layer="96" rot="R90"/>
 </instance>
-<instance part="+3V1" gate="G$1" x="72.39" y="74.93" smashed="yes">
-<attribute name="VALUE" x="69.85" y="69.85" size="1.778" layer="96" rot="R90"/>
-</instance>
-<instance part="GND1" gate="1" x="72.39" y="50.8" smashed="yes">
-<attribute name="VALUE" x="69.85" y="48.26" size="1.778" layer="96"/>
+<instance part="+3V1" gate="G$1" x="71.12" y="76.2" smashed="yes">
+<attribute name="VALUE" x="68.58" y="71.12" size="1.778" layer="96" rot="R90"/>
+</instance>
+<instance part="GND1" gate="1" x="71.12" y="50.8" smashed="yes">
+<attribute name="VALUE" x="68.58" y="48.26" size="1.778" layer="96"/>
 </instance>
 <instance part="R2" gate="G$1" x="143.51" y="77.47" smashed="yes" rot="R90">
@@
 <instance part="+3V7" gate="G$1" x="69.85" y="108.712" smashed="yes">
 <attribute name="VALUE" x="67.31" y="103.632" size="1.778" layer="96" rot="R90"/>
+</instance>
+<instance part="C5" gate="G$1" x="71.12" y="63.5" smashed="yes">
+<attribute name="NAME" x="72.136" y="64.135" size="1.778" layer="95"/>
+<attribute name="VALUE" x="72.136" y="59.309" size="1.778" layer="96"/>
+</instance>
+<instance part="C6" gate="G$1" x="119.38" y="22.86" smashed="yes">
+<attribute name="NAME" x="120.396" y="23.495" size="1.778" layer="95"/>
+<attribute name="VALUE" x="120.396" y="18.669" size="1.778" layer="96"/>
 </instance>
 </instances>
@@
 <segment>
 <pinref part="U$1" gate="G$1" pin="VCC"/>
-<wire x1="76.2" y1="68.58" x2="72.39" y2="68.58" width="0.1524" layer="91"/>
-<wire x1="72.39" y1="68.58" x2="72.39" y2="72.39" width="0.1524" layer="91"/>
+<wire x1="76.2" y1="68.58" x2="71.12" y2="68.58" width="0.1524" layer="91"/>
+<wire x1="71.12" y1="68.58" x2="71.12" y2="73.66" width="0.1524" layer="91"/>
 <pinref part="+3V1" gate="G$1" pin="+3V3"/>
+<pinref part="C5" gate="G$1" pin="1"/>
+<wire x1="71.12" y1="66.04" x2="71.12" y2="68.58" width="0.1524" layer="91"/>
+<junction x="71.12" y="68.58"/>
 </segment>
 <segment>
@@
 <segment>
 <pinref part="GND1" gate="1" pin="GND"/>
-<wire x1="72.39" y1="53.34" x2="72.39" y2="55.88" width="0.1524" layer="91"/>
+<wire x1="71.12" y1="53.34" x2="71.12" y2="55.88" width="0.1524" layer="91"/>
 <pinref part="U$1" gate="G$1" pin="GND"/>
-<wire x1="72.39" y1="55.88" x2="76.2" y2="55.88" width="0.1524" layer="91"/>
+<wire x1="71.12" y1="55.88" x2="76.2" y2="55.88" width="0.1524" layer="91"/>
+<pinref part="C5" gate="G$1" pin="2"/>
+<wire x1="71.12" y1="58.42" x2="71.12" y2="55.88" width="0.1524" layer="91"/>
+<junction x="71.12" y="55.88"/>
 </segment>
 <segment>
@@
 <wire x1="132.08" y1="19.05" x2="132.08" y2="15.24" width="0.1524" layer="91"/>
 <pinref part="GND4" gate="1" pin="GND"/>
+<wire x1="132.08" y1="15.24" x2="119.38" y2="15.24" width="0.1524" layer="91"/>
+<junction x="132.08" y="15.24"/>
+<pinref part="C6" gate="G$1" pin="2"/>
+<wire x1="119.38" y1="15.24" x2="119.38" y2="17.78" width="0.1524" layer="91"/>
 </segment>
 <segment>
@@
 <net name="CURRENT" class="0">
 <segment>
-<pinref part="U$1" gate="G$1" pin="PB3/XTAL1/CLKI/ADC3"/>
-<wire x1="127" y1="60.96" x2="132.08" y2="60.96" width="0.1524" layer="91"/>
-<label x="132.08" y="60.96" size="1.27" layer="95" xref="yes"/>
-</segment>
-<segment>
 <pinref part="R6" gate="G$1" pin="1"/>
 <wire x1="35.56" y1="59.69" x2="40.64" y2="59.69" width="0.1524" layer="91"/>
@@
 <label x="40.64" y="59.69" size="1.27" layer="95" xref="yes"/>
 </segment>
-</net>
-<net name="TEMPERATURE" class="0">
 <segment>
 <pinref part="U$1" gate="G$1" pin="PB4/XTAL2/CLKO/ADC2"/>
@@
 <label x="132.08" y="58.42" size="1.27" layer="95" xref="yes"/>
 </segment>
+</net>
+<net name="TEMPERATURE" class="0">
 <segment>
 <pinref part="THERMISTOR" gate="G$1" pin="2"/>
 <wire x1="143.51" y1="35.56" x2="132.08" y2="35.56" width="0.1524" layer="91"/>
-<wire x1="132.08" y1="35.56" x2="132.08" y2="29.21" width="0.1524" layer="91"/>
+<wire x1="132.08" y1="35.56" x2="132.08" y2="30.48" width="0.1524" layer="91"/>
 <pinref part="R5" gate="G$1" pin="2"/>
 <label x="132.08" y="35.56" size="1.27" layer="95" rot="R180" xref="yes"/>
+<pinref part="C6" gate="G$1" pin="1"/>
+<wire x1="132.08" y1="30.48" x2="132.08" y2="29.21" width="0.1524" layer="91"/>
+<wire x1="119.38" y1="25.4" x2="119.38" y2="30.48" width="0.1524" layer="91"/>
+<wire x1="119.38" y1="30.48" x2="132.08" y2="30.48" width="0.1524" layer="91"/>
+<junction x="132.08" y="30.48"/>
+</segment>
+<segment>
+<pinref part="U$1" gate="G$1" pin="PB3/XTAL1/CLKI/ADC3"/>
+<wire x1="127" y1="60.96" x2="132.08" y2="60.96" width="0.1524" layer="91"/>
+<label x="132.08" y="60.96" size="1.27" layer="95" xref="yes"/>
 </segment>
 </net>
@@
 </segment>
 </net>
-<net name="M-IP+" class="0">
+<net name="M-IP+" class="1">
 <segment>
 <pinref part="U$4" gate="G$1" pin="V-"/>
@@
 </segment>
 </net>
-<net name="M-IP-" class="0">
+<net name="M-IP-" class="1">
 <segment>
 <pinref part="U$2" gate="G$1" pin="IP-"/>
@@
 </segment>
 </net>
-<net name="M+" class="0">
+<net name="M+" class="1">
 <segment>
 <pinref part="U$5" gate="G$1" pin="V+"/>
