File: currentsense.brd (EAGLE design)
At the start: 78.7 x 70.8 mm, 18 parts

Commit message: more layout work
Parts:
- moved R1 42.6 mm to (72.9, 9.78), turned to 90 degrees
- moved ISP 41.9 mm to (67.3, 5.08)
- moved U$1 37.0 mm to (53.3, 4.95), turned to 90 degrees
- moved R3 30.5 mm to (45.7, 2.54), turned to 0 degrees
- moved R2 29.2 mm to (45.7, 7.62), turned to 0 degrees
- moved U$4 27.4 mm to (49.5, 39.4)
- moved R5 25.7 mm to (62.5, 9.78), turned to 90 degrees
- moved U$5 23.9 mm to (24.1, 39.4)
- moved THERMISTOR 20.4 mm to (67.4, 15.5), turned to 180 degrees
- moved DATA 17.8 mm to (33.0, 5.08)
- moved R6 15.7 mm to (41.7, 13.7)
- moved C1 15.3 mm to (37.0, 12.7)
- moved C2 14.2 mm to (32.1, 13.8)
- moved U$2 13.6 mm to (36.8, 18.4)
- moved U$3 10.2 mm to (15.2, 12.7), turned to 270 degrees
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Connections:
- net N$1 renamed M-IP+
- net N$3 renamed M-IP-
- net N$4 renamed M+
- removed net OC_DETECT: DATA.3
- removed net SDA: DATA.1
- net OC_DETECT/6: now also DATA.2
- net SCL/7: now also DATA.3; no longer DATA.2
- net SDA/5: now also DATA.1
Routing:
- net M-IP+: track 40.6 -> 0.00 mm, vias 0 -> 2
- net M-IP-: track 31.8 -> 0.00 mm, vias 0 -> 2
- added copper zone on layer 1, net M+
- added copper zone on layer 16, net M+
- added copper zone on layer 1, net M-IP+
- added copper zone on layer 16, net M-IP+
- added copper zone on layer 1, net M-IP-
- added copper zone on layer 16, net M-IP-
Other:
- board size 78.7 x 70.8 mm -> 86.3 x 56.8 mm

Commit message: add board files
Parts:
- added C5, C6: 0.1uF, rcl:C0805
- C1, C2: value (none) -> 0.1uF
- C3, C4: value (none) -> 10uF
- R2, R3: value (none) -> 10k
- R6: value (none) -> 2.2k
- moved R3 15.7 mm to (30.5, 6.35), turned to 90 degrees
- moved U$1 7.00 mm to (59.8, 7.62), turned to 180 degrees
- moved R1 6.84 mm to (79.2, 12.3)
- moved C1 6.48 mm to (43.3, 14.0)
- moved R6 6.48 mm to (48.0, 15.0)
- moved ISP 6.38 mm to (73.7, 5.71), turned to 270 degrees
- moved THERMISTOR 6.35 mm to (73.8, 15.5)
- moved C3 6.35 mm to (19.1, 5.08)
- moved U$2 6.35 mm to (43.2, 18.4)
- moved U$4 6.35 mm to (55.9, 39.4)
- moved U$5 6.35 mm to (30.5, 39.4)
- moved C4 6.35 mm to (10.2, 14.0)
- moved POWER 6.35 mm to (7.62, 5.08)
- moved U$3 6.35 mm to (21.6, 12.7)
- moved DATA 6.35 mm to (39.4, 5.08), turned to 180 degrees
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Connections:
- net +3V3: now also C5.1
- net CURRENT: now also U$1.3; no longer U$1.2
- net GND: now also C5.2, C6.2
- net TEMPERATURE: now also C6.1, U$1.2; no longer U$1.3
Routing:
- net +3V3: track 0.00 -> 105.9 mm
- net SCL/7: track 0.00 -> 47.9 mm
- net SDA/5: track 0.00 -> 45.8 mm, vias 0 -> 2
- net OC_DETECT/6: track 0.00 -> 38.8 mm, vias 0 -> 2
- net RESET: track 0.00 -> 31.1 mm, vias 0 -> 1
- net VCC: track 0.00 -> 17.9 mm
- net CURRENT: track 0.00 -> 17.1 mm
- net TEMPERATURE: track 0.00 -> 15.3 mm
- net N$2: track 0.00 -> 4.22 mm
- added copper zone on layer 1, net GND
- added copper zone on layer 16, net GND
- added copper zone on layer 15, net M+
- added copper zone on layer 2, net M+
- added copper zone on layer 15, net M-IP+
- added copper zone on layer 2, net M-IP+
- added copper zone on layer 15, net M-IP-
- added copper zone on layer 2, net M-IP-
Other:
- board text added: "*"

Commit message: minor error
Other:
- board text added: "* * . ' .* . . * Current Sense Board v0 . Giselle Koo . * * For CU Robotic Mining Team * . * . * . ' . *."
Changed lines of the file:
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@@
 <setting verticaltext="up"/>
 </settings>
-<grid distance="50" unitdist="mil" unit="inch" style="lines" multiple="1" display="no" altdistance="0.025" altunitdist="inch" altunit="mil"/>
+<grid distance="50" unitdist="mil" unit="mil" style="lines" multiple="1" display="no" altdistance="0.025" altunitdist="inch" altunit="mil"/>
 <layers>
 <layer number="1" name="Top" color="4" fill="1" visible="yes" active="yes"/>
-<layer number="2" name="Route2" color="16" fill="1" visible="no" active="yes"/>
+<layer number="2" name="Route2" color="16" fill="1" visible="yes" active="yes"/>
 <layer number="3" name="Route3" color="17" fill="1" visible="no" active="no"/>
 <layer number="4" name="Route4" color="18" fill="1" visible="no" active="no"/>
@@
 <layer number="27" name="tValues" color="7" fill="1" visible="no" active="yes"/>
 <layer number="28" name="bValues" color="7" fill="1" visible="no" active="yes"/>
-<layer number="29" name="tStop" color="7" fill="3" visible="yes" active="yes"/>
-<layer number="30" name="bStop" color="7" fill="6" visible="yes" active="yes"/>
+<layer number="29" name="tStop" color="7" fill="3" visible="no" active="yes"/>
+<layer number="30" name="bStop" color="7" fill="6" visible="no" active="yes"/>
 <layer number="31" name="tCream" color="7" fill="4" visible="no" active="yes"/>
 <layer number="32" name="bCream" color="7" fill="5" visible="no" active="yes"/>
@@
 <layer number="43" name="vRestrict" color="2" fill="10" visible="no" active="yes"/>
 <layer number="44" name="Drills" color="7" fill="1" visible="no" active="yes"/>
-<layer number="45" name="Holes" color="7" fill="1" visible="yes" active="yes"/>
+<layer number="45" name="Holes" color="7" fill="1" visible="no" active="yes"/>
 <layer number="46" name="Milling" color="3" fill="1" visible="no" active="yes"/>
 <layer number="47" name="Measures" color="7" fill="1" visible="no" active="yes"/>
@@
 <hole x="82.55" y="27.94" drill="3.2"/>
 <text x="70.485" y="8.255" size="1.778" layer="21">*</text>
+<text x="40.64" y="15.24" size="1.778" layer="22" rot="MR0" align="center">*
+*     . '       .*      .
+.  * Current Sense Board v0
+.    Giselle Koo . *
+*  For CU Robotic Mining Team *
+ .       *  .        * .       '
+.    *.</text>
 </plain>
 <attributes>
@@
 </classes>
 <designrules name="advanced-circuits-4layer *">
-<description language="en">&lt;b&gt;OSH Park Design Rules&lt;/b&gt;
-&lt;p&gt;
-Please make sure your boards conform to these design rules.
-&lt;/p&gt;
-&lt;p&gt;
-Note, that not all DRC settings must be set by the manufacturer. Several can be adjusted for the design, including those listed on our docs page here.
-&lt;a href=&quot;http://docs.oshpark.com/design-tools/eagle/design-rules-files/&quot;&gt;Adjustable Settings&lt;/a&gt;
-&lt;/p&gt;</description>
+<description language="en">&lt;B&gt;Advanced Circuits (4pcb.com) &lt;/B&gt;&lt;br&gt;
+Adapted from OSH Park 4 layer Design rules</description>
 <param name="layerSetup" value="(1*2*15*16)"/>
 <param name="mtCopper" value="0.035559375mm 0.035559375mm 0.0356mm 0.0356mm 0.0356mm 0.0356mm 0.0356mm 0.0356mm 0.0356mm 0.0356mm 0.0356mm 0.0356mm 0.0356mm 0.0356mm 0.035559375mm 0.035559375mm"/>
@@
 </element>
 <element name="THERMISTOR" library="pinhead" library_urn="urn:adsk.eagle:library:325" package="1X02" package3d_urn="urn:adsk.eagle:package:22435/2" value="" x="73.787" y="15.494" smashed="yes" rot="R180">
-<attribute name="NAME" x="76.4032" y="13.6652" size="1.27" layer="25" ratio="10" rot="R180"/>
+<attribute name="NAME" x="78.9432" y="18.7452" size="1.27" layer="25" ratio="10" rot="R180"/>
 <attribute name="POPULARITY" value="98" x="28.067" y="59.944" size="1.778" layer="27" rot="R180" display="off"/>
 <attribute name="VALUE" x="76.327" y="18.669" size="1.27" layer="27" rot="R180"/>
@@
 <element name="U$5" library="XT Connectors" package="XT60_RA" value="XT60-RA" x="30.48" y="39.37" smashed="yes" rot="R270"/>
 <element name="U$3" library="currentlim" package="SOT223" value="LM1117" x="21.59" y="12.7" smashed="yes" rot="R270">
-<attribute name="NAME" x="21.6408" y="15.24" size="1.27" layer="25" rot="R270"/>
+<attribute name="NAME" x="20.32" y="16.5608" size="1.27" layer="25"/>
 <attribute name="VALUE" x="20.2692" y="15.24" size="1.27" layer="27" rot="R270"/>
 </element>
@@
 <contactref element="U$1" pad="2"/>
 <wire x1="60.462" y1="10.774" x2="60.462" y2="12.837" width="0.508" layer="1"/>
-<wire x1="60.462" y1="12.837" x2="60.96" y2="13.335" width="0.508" layer="1"/>
 <wire x1="67.564" y1="13.269" x2="69.789" y2="15.494" width="0.508" layer="1"/>
 <wire x1="69.789" y1="15.494" x2="72.517" y2="15.494" width="0.508" layer="1"/>
 <contactref element="C6" pad="1"/>
-<wire x1="60.96" y1="13.335" x2="67.498" y2="13.335" width="0.508" layer="1"/>
-<wire x1="67.498" y1="13.335" x2="67.564" y2="13.269" width="0.508" layer="1"/>
-<wire x1="67.564" y1="13.269" x2="63.5" y2="13.655" width="0" layer="19" extent="1-1"/>
+<wire x1="61.28" y1="13.655" x2="63.5" y2="13.655" width="0.508" layer="1"/>
+<wire x1="60.462" y1="12.837" x2="61.28" y2="13.655" width="0.508" layer="1"/>
+<wire x1="63.5" y1="13.655" x2="67.178" y2="13.655" width="0.508" layer="1"/>
+<wire x1="67.178" y1="13.655" x2="67.564" y2="13.269" width="0.508" layer="1"/>
 </signal>
 <signal name="RESET">
@@
 </polygon>
 <polygon width="0" layer="2" thermals="no">
-<vertex x="80.01" y="38.735"/>
-<vertex x="37.338" y="38.735"/>
-<vertex x="37.338" y="22.225"/>
-<vertex x="80.01" y="22.225"/>
+<vertex x="86.36" y="38.735"/>
+<vertex x="43.688" y="38.735"/>
+<vertex x="43.688" y="22.225"/>
+<vertex x="86.36" y="22.225"/>
 </polygon>
 </signal>
@@
 <via x="26.67" y="24.765" extent="1-16" drill="0.508"/>
 <polygon width="0" layer="2" thermals="no">
-<vertex x="-6.35" y="38.735"/>
-<vertex x="36.322" y="38.735"/>
-<vertex x="36.322" y="22.225"/>
-<vertex x="-6.35" y="22.225"/>
+<vertex x="0" y="38.735"/>
+<vertex x="42.672" y="38.735"/>
+<vertex x="42.672" y="22.225"/>
+<vertex x="0" y="22.225"/>
 </polygon>
 <polygon width="0" layer="15" thermals="no">
@@
 </polygon>
 <polygon width="0" layer="2" thermals="no">
-<vertex x="-6.35" y="55.88"/>
-<vertex x="-6.35" y="40.005"/>
-<vertex x="80.01" y="40.005"/>
-<vertex x="80.01" y="55.88"/>
+<vertex x="0" y="55.88"/>
+<vertex x="0" y="40.005"/>
+<vertex x="86.36" y="40.005"/>
+<vertex x="86.36" y="55.88"/>
 </polygon>
 </signal>
@@
 </drawing>
 <compatibility>
+<note version="6.3" minversion="6.2.2" severity="warning">
+Since Version 6.2.2 text objects can contain more than one line,
+which will not be processed correctly with this version.
+</note>
 <note version="8.2" severity="warning">
 Since Version 8.2, EAGLE supports online libraries. The ids
